File: Jorge/Jorge.kicad_sch (KiCad schematic)
At the start: 9 parts

Commit message: Modified PCB to user Battery 12V -> Regulator 6V -> ESP32 regulator 3.3V system
Parts:
- BMP1: footprint Ernest:BME280_breakout_footprint -> Jorge:BME280_breakout_footprint
- GY-GPS6MV1: footprint Ernest:GY-GPS6MV2_footprint -> Jorge:GY-GPS6MV2_footprint
- MP1584EN1: footprint Ernest:MP1584_breakout_footprint -> Jorge:MP1584_breakout_footprint
- MPU-1: footprint Ernest:MPU6050_breakout_footprint -> Jorge:MPU6050_breakout_footprint
- TB1: footprint Ernest:TB6612_breakout_footprint -> Jorge:TB6612_breakout_footprint
- U1: symbol Esp32s-38-pin Dev Board:Esp32 -> ESP32-38pin:Esp32
Connections:
- net +3.3V: no longer MP1584EN1.3 (OUT_VCC), SG1.2 (VCC)
- net GND: now also U1.32 (GND)
- net +6V: now reaches U1.19 (5V)
- net +6V: now also MP1584EN1.3 (OUT_VCC), SG1.2 (VCC)
- no-connect marks 37 -> 35
