File: Electronics/Jorge/Jorge.kicad_pcb (KiCad board)
At the start: 2 copper layers, 9 parts

Commit message: Working Aleph v0.1 Project
Parts:
- renumbered SG1 to MG996R
Other:
- board outline added: 57 x 115 mm
Changed lines of the file:
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@@
 			(plot_on_all_layers_selection 0x00000000_00000000_00000000_00000000)
 			(disableapertmacros no)
-			(usegerberextensions no)
+			(usegerberextensions yes)
 			(usegerberattributes yes)
 			(usegerberadvancedattributes yes)
@@
 			(dashed_line_gap_ratio 3.000000)
 			(svgprecision 4)
-			(plotframeref no)
+			(plotframeref yes)
 			(mode 1)
 			(useauxorigin no)
@@
 			(sketchdnponfab yes)
 			(crossoutdnponfab yes)
-			(subtractmaskfromsilk no)
+			(subtractmaskfromsilk yes)
 			(outputformat 1)
 			(mirror no)
-			(drillshape 1)
+			(drillshape 0)
 			(scaleselection 1)
-			(outputdirectory "")
+			(outputdirectory "gerbers/")
 		)
 	)
@@
 		(descr "Through hole straight socket strip, 1x03, 2.54mm pitch, single row (from Kicad 4.0.7), script generated")
 		(tags "Through hole socket strip THT 1x03 2.54mm single row")
-		(property "Reference" "SG1"
+		(property "Reference" "MG996R"
 			(at 2.975 2.54 180)
 			(layer "F.SilkS")
@@
 		(stroke
 			(width 0.05)
-			(type default)
+			(type solid)
 		)
 		(fill no)
-		(layer "B.CrtYd")
+		(layer "Edge.Cuts")
 	)
 	(gr_text "↑"
